Commit message: hardware testing 25-9 1

File: legged_examples/legged_unitree/legged_unitree_description/urdf/jamal/const.xacro (robot description, xacro)
@@ -65,5 +65,5 @@
     <!-- trunk -->
     <xacro:property name="trunk_mass" value="12.8185384756311"/>
-    <xacro:property name="trunk_com_x" value="0"/>
+    <xacro:property name="trunk_com_x" value="0.05"/>
     <xacro:property name="trunk_com_y" value="0"/>
     <xacro:property name="trunk_com_z" value="-0.0005"/>

Commit message: hardware testing 28-9 1

File: legged_examples/legged_unitree/legged_unitree_description/urdf/jamal/const.xacro (robot description, xacro)
@@ -22,5 +22,6 @@
     <xacro:property name="thigh_offset" value="0.08"/>
     <xacro:property name="thigh_length" value="0.225"/>
-    <xacro:property name="calf_length" value="0.235"/>
+    <!-- <xacro:property name="calf_length" value="0.235"/> -->
+    <xacro:property name="calf_length" value="0.250"/>
     <!-- leg offset from trunk center value -->
     <xacro:property name="leg_offset_x" value="0.26209"/>

Commit message: hardware testing 28-9 3

File: legged_examples/legged_unitree/legged_unitree_description/urdf/jamal/const.xacro (robot description, xacro)
@@ -66,5 +66,5 @@
     <!-- trunk -->
     <xacro:property name="trunk_mass" value="12.8185384756311"/>
-    <xacro:property name="trunk_com_x" value="0.05"/>
+    <xacro:property name="trunk_com_x" value="-0.07"/>
     <xacro:property name="trunk_com_y" value="0"/>
     <xacro:property name="trunk_com_z" value="-0.0005"/>
@@ -77,7 +77,10 @@
     <!-- hip (left front) -->
     <xacro:property name="hip_mass" value="0.933762854916433"/>
-    <xacro:property name="hip_com_x" value="-0.005657"/>
+    <!-- <xacro:property name="hip_com_x" value="-0.005657"/>
     <xacro:property name="hip_com_y" value="-0.008752"/>
-    <xacro:property name="hip_com_z" value="-0.000102"/>
+    <xacro:property name="hip_com_z" value="-0.000102"/> -->
+    <xacro:property name="hip_com_x" value="0.0"/>
+    <xacro:property name="hip_com_y" value="0.0"/>
+    <xacro:property name="hip_com_z" value="0.0"/>
     <xacro:property name="hip_ixx" value="0.000832273911083319"/>
     <xacro:property name="hip_ixy" value="2.01742652907359E-06"/>
@@ -88,7 +91,10 @@
     <!-- thigh -->
     <xacro:property name="thigh_mass" value="1.32134262348697"/>
-    <xacro:property name="thigh_com_x" value="-0.003342"/>
+    <!-- <xacro:property name="thigh_com_x" value="-0.003342"/>
     <xacro:property name="thigh_com_y" value="-0.018054"/>
-    <xacro:property name="thigh_com_z" value="-0.033451"/>
+    <xacro:property name="thigh_com_z" value="-0.033451"/> -->
+    <xacro:property name="thigh_com_x" value="0.0"/>
+    <xacro:property name="thigh_com_y" value="0.0"/>
+    <xacro:property name="thigh_com_z" value="0.0"/>
     <xacro:property name="thigh_ixx" value="0.00262880898900224"/>
     <xacro:property name="thigh_ixy" value="3.0753036678596E-07"/>
@@ -99,7 +105,10 @@
     <!-- calf -->
     <xacro:property name="calf_mass" value="0.12879265462489"/>
-    <xacro:property name="calf_com_x" value="0.006197"/>
+    <!-- <xacro:property name="calf_com_x" value="0.006197"/>
     <xacro:property name="calf_com_y" value="0.001408"/>
-    <xacro:property name="calf_com_z" value="-0.116695"/>
+    <xacro:property name="calf_com_z" value="-0.116695"/> -->
+    <xacro:property name="calf_com_x" value="0.0"/>
+    <xacro:property name="calf_com_y" value="0.0"/>
+    <xacro:property name="calf_com_z" value="0.0"/>
     <xacro:property name="calf_ixx" value="0.000445341853265945"/>
     <xacro:property name="calf_ixy" value="-7.71823686634482E-09"/>
