Commit message: hardware testing 30-9 1

File: legged_examples/legged_unitree/legged_unitree_description/urdf/common/leg.xacro (robot description, xacro)
@@ -78,5 +78,6 @@
             </visual>
             <collision>
-                <origin rpy="0 ${pi/2.0+0.1} 0" xyz="${thigh_x_offset} 0 ${-thigh_length/2.0}"/>
+                <!-- <origin rpy="0 ${pi/2.0+0.1} 0" xyz="${thigh_x_offset} 0 ${-thigh_length/2.0}"/> -->
+                <origin rpy="0 ${pi/2.0} 0" xyz="${thigh_x_offset} 0 ${-thigh_length/2.0}"/>
                 <geometry>
                     <box size="${thigh_length} ${thigh_width} ${thigh_height}"/>
@@ -108,5 +109,6 @@
         <link name="${prefix}_calf">
             <visual>
-                <origin rpy="0 0.06 0" xyz="0 0 0"/>
+                <!-- <origin rpy="0 0.06 0" xyz="0 0 0"/> -->
+                <origin rpy="0 0 0" xyz="0 0 0"/>
                 <geometry>
                     <mesh filename="${mesh_path}/calf.dae"

File: legged_examples/legged_unitree/legged_unitree_description/urdf/jamal/const.xacro (robot description, xacro)
@@ -14,5 +14,6 @@
     <xacro:property name="thigh_width" value="0.0245"/>
     <xacro:property name="thigh_height" value="0.034"/>
-    <xacro:property name="thigh_x_offset" value="-0.015"/>
+    <!-- <xacro:property name="thigh_x_offset" value="-0.015"/> -->
+    <xacro:property name="thigh_x_offset" value="0.0"/>
     <xacro:property name="calf_width" value="0.016"/>
     <xacro:property name="calf_height" value="0.016"/>
@@ -20,15 +21,15 @@
     <xacro:property name="foot_radius" value="0.017"/>
     <!-- kinematic value -->
-    <xacro:property name="thigh_offset" value="0.08"/>
+    <xacro:property name="thigh_offset" value="0.10755"/>
     <xacro:property name="thigh_length" value="0.225"/>
     <!-- <xacro:property name="calf_length" value="0.235"/> -->
     <xacro:property name="calf_length" value="0.250"/>
     <!-- leg offset from trunk center value -->
-    <xacro:property name="leg_offset_x" value="0.26209"/>
-    <xacro:property name="leg_offset_y" value="0.08013"/>
+    <xacro:property name="leg_offset_x" value="0.2699"/>
+    <xacro:property name="leg_offset_y" value="0.08028"/>
     <!-- <xacro:property name="trunk_offset_z" value="0.01675"/> -->
     <xacro:property name="hip_offset" value="0.0"/>
     <!-- offset of link and rotor locations (left front) -->
-    <xacro:property name="hip_offset_x" value="0.1881"/>
+    <!-- <xacro:property name="hip_offset_x" value="0.1881"/>
     <xacro:property name="hip_offset_y" value="0.04675"/>
     <xacro:property name="hip_offset_z" value="0.0"/>
@@ -47,4 +48,23 @@
     <xacro:property name="calf_rotor_offset_x" value="0.0"/>
     <xacro:property name="calf_rotor_offset_y" value="-0.03235"/>
+    <xacro:property name="calf_rotor_offset_z" value="0.0"/> -->
+    <!-- offset of link and rotor locations (left front) -->
+    <xacro:property name="hip_offset_x" value="0.2699"/>
+    <xacro:property name="hip_offset_y" value="0.08028"/>
+    <xacro:property name="hip_offset_z" value="0.0"/>
+    <xacro:property name="hip_rotor_offset_x" value="0.2119"/>
+    <xacro:property name="hip_rotor_offset_y" value="0.08028"/>
+    <xacro:property name="hip_rotor_offset_z" value="0.0"/>
+    <xacro:property name="thigh_offset_x" value="0"/>
+    <xacro:property name="thigh_offset_y" value="0.10755"/>
+    <xacro:property name="thigh_offset_z" value="0.0"/>
+    <xacro:property name="thigh_rotor_offset_x" value="0.0"/>
+    <xacro:property name="thigh_rotor_offset_y" value="-0.0295"/>
+    <xacro:property name="thigh_rotor_offset_z" value="0.0"/>
+    <xacro:property name="calf_offset_x" value="0.0"/>
+    <xacro:property name="calf_offset_y" value="0.0"/>
+    <xacro:property name="calf_offset_z" value="-0.225"/>
+    <xacro:property name="calf_rotor_offset_x" value="0.0"/>
+    <xacro:property name="calf_rotor_offset_y" value="0.0"/>
     <xacro:property name="calf_rotor_offset_z" value="0.0"/>
     <!-- joint limits -->
@@ -53,20 +73,21 @@
     <xacro:property name="hip_position_max" value="0.863"/>
     <xacro:property name="hip_position_min" value="-0.863"/>
-    <xacro:property name="hip_velocity_max" value="30.1"/>
+    <xacro:property name="hip_velocity_max" value="8"/>
     <xacro:property name="hip_torque_max" value="48"/>
     <xacro:property name="thigh_position_max" value="4.501"/>
     <xacro:property name="thigh_position_min" value="-0.686"/>
-    <xacro:property name="thigh_velocity_max" value="30.1"/>
+    <xacro:property name="thigh_velocity_max" value="8"/>
     <xacro:property name="thigh_torque_max" value="48"/>
     <xacro:property name="calf_position_max" value="-0.888"/>
     <xacro:property name="calf_position_min" value="-2.818"/>
-    <xacro:property name="calf_velocity_max" value="20.06"/>
+    <xacro:property name="calf_velocity_max" value="8"/>
     <xacro:property name="calf_torque_max" value="48"/>
     <!-- dynamics inertial value        total 12.84kg -->
     <!-- trunk -->
     <xacro:property name="trunk_mass" value="12.8185384756311"/>
-    <xacro:property name="trunk_com_x" value="-0.07"/>
+    <xacro:property name="trunk_com_x" value="0.03"/>
     <xacro:property name="trunk_com_y" value="0"/>
-    <xacro:property name="trunk_com_z" value="-0.0005"/>
+    <!-- <xacro:property name="trunk_com_z" value="-0.0005"/> -->
+    <xacro:property name="trunk_com_z" value="0.0"/>
     <xacro:property name="trunk_ixx" value="0.0565667940678376"/>
     <xacro:property name="trunk_ixy" value="-8.54731557026013E-06"/>
